File: electronics/view_base/view_base - Copy.kicad_pcb (KiCad board)
At the start: 4 copper layers, 81.2 x 81.2 mm, 259 parts, among them J1 USB_C_Receptacle_USB2.0, J2 A, J3 B, J4 LCD, J5 59453-081110EDHLF, J6 BLDC, J7 SM04B-SRSS-TB(LF)(SN), J8 SM04B-SRSS-TB(LF)(SN), J9 SM04B-SRSS-TB(LF)(SN), Q1 MMBT4403, Q2 BSS138, Q3 BSS138, SW1 RST, SW2 Boot, U1 SN74LV1T34DBV, U10 LP5907MFX-2.8, U11 ESP32-S3-WROOM-1U-N16R8, U2 MT6701-CT, U3 VEML7700, U4 AMS1117-3.3, U5 USBLC6-2SC6, U6 HX711, U8 TMC6300, U9 VL53L0CXV0DH_1

Commit message: Layout battery controller and fuel gauge
Parts:
- removed TP12: RX, cleaned footprints:TestPoint_Pad_D2.0mm_ValueSilk
- removed TP13: TX, cleaned footprints:TestPoint_Pad_D2.0mm_ValueSilk
- removed TP17: IO40, cleaned footprints:TestPoint_Pad_D2.0mm_ValueSilk
- removed TP18: IO41, cleaned footprints:TestPoint_Pad_D2.0mm_ValueSilk
- removed TP19: IO42, cleaned footprints:TestPoint_Pad_D2.0mm_ValueSilk
- removed TP20: IO45, cleaned footprints:TestPoint_Pad_D2.0mm_ValueSilk
- removed TP21: IO46, cleaned footprints:TestPoint_Pad_D2.0mm_ValueSilk
- removed TP22: IO47, cleaned footprints:TestPoint_Pad_D2.0mm_ValueSilk
- removed TP23: IO48, cleaned footprints:TestPoint_Pad_D2.0mm_ValueSilk
- added TP24: IO40, TestPoint:TestPoint_Pad_D2.0mm, B.Cu at (162.2, 138.2)
- added TP25: IO41, TestPoint:TestPoint_Pad_D2.0mm, B.Cu at (159.2, 138.2)
- added TP26: IO42, TestPoint:TestPoint_Pad_D2.0mm, B.Cu at (156.2, 138.2)
- added TP27: IO45, TestPoint:TestPoint_Pad_D2.0mm, B.Cu at (165.2, 138.2)
- added TP28: IO46, TestPoint:TestPoint_Pad_D2.0mm, B.Cu at (174.2, 138.2)
- added TP29: IO47, TestPoint:TestPoint_Pad_D2.0mm, B.Cu at (171.2, 138.2)
- added TP30: IO48, TestPoint:TestPoint_Pad_D2.0mm, B.Cu at (168.2, 138.2)
- added TP31: RX, TestPoint:TestPoint_Pad_D2.0mm, B.Cu at (117.8, 138.2)
- added TP32: TX, TestPoint:TestPoint_Pad_D2.0mm, B.Cu at (113.8, 138.2)
Routing:
- net Net-(U7-IO46): track 104.6 -> 0.00 mm, vias 2 -> 0
- net Net-(U11-IO46): track 0.00 -> 104.6 mm, vias 0 -> 1
- net Net-(U7-IO47): track 93.0 -> 0.00 mm, vias 2 -> 0
- net Net-(U11-IO47): track 0.00 -> 93.0 mm, vias 0 -> 1
- net Net-(U7-IO48): track 91.2 -> 0.00 mm, vias 2 -> 0
- net Net-(U11-IO48): track 0.00 -> 91.2 mm
- net Net-(U7-IO45): track 87.4 -> 0.00 mm, vias 2 -> 0
- net Net-(U11-IO45): track 0.00 -> 87.4 mm, vias 0 -> 1
- net Net-(U7-IO40): track 76.1 -> 0.00 mm, vias 2 -> 0
- net Net-(U11-IO40): track 0.00 -> 76.1 mm, vias 0 -> 1
- net Net-(U7-IO41): track 72.2 -> 0.00 mm, vias 2 -> 0
- net Net-(U11-IO41): track 0.00 -> 72.2 mm, vias 0 -> 2
- net Net-(U7-IO42): track 68.0 -> 0.00 mm, vias 2 -> 0
- net Net-(U11-IO42): track 0.00 -> 68.0 mm, vias 0 -> 2
- net (no net): vias 0 -> 6

Commit message: Initial commit
Parts:
- removed TP24: IO40, TestPoint:TestPoint_Pad_D2.0mm
- removed TP25: IO41, TestPoint:TestPoint_Pad_D2.0mm
- removed TP26: IO42, TestPoint:TestPoint_Pad_D2.0mm
- removed TP27: IO45, TestPoint:TestPoint_Pad_D2.0mm
- removed TP28: IO46, TestPoint:TestPoint_Pad_D2.0mm
- removed TP29: IO47, TestPoint:TestPoint_Pad_D2.0mm
- removed TP30: IO48, TestPoint:TestPoint_Pad_D2.0mm
- removed TP31: RX, TestPoint:TestPoint_Pad_D2.0mm
- removed TP32: TX, TestPoint:TestPoint_Pad_D2.0mm
- added TP12: RX, cleaned footprints:TestPoint_Pad_D2.0mm_ValueSilk, B.Cu at (117.8, 138.2)
- added TP13: TX, cleaned footprints:TestPoint_Pad_D2.0mm_ValueSilk, B.Cu at (113.8, 138.2)
- added TP17: IO40, cleaned footprints:TestPoint_Pad_D2.0mm_ValueSilk, B.Cu at (162.2, 138.2)
- added TP18: IO41, cleaned footprints:TestPoint_Pad_D2.0mm_ValueSilk, B.Cu at (159.2, 138.2)
- added TP19: IO42, cleaned footprints:TestPoint_Pad_D2.0mm_ValueSilk, B.Cu at (156.2, 138.2)
- added TP20: IO45, cleaned footprints:TestPoint_Pad_D2.0mm_ValueSilk, B.Cu at (165.2, 138.2)
- added TP21: IO46, cleaned footprints:TestPoint_Pad_D2.0mm_ValueSilk, B.Cu at (174.2, 138.2)
- added TP22: IO47, cleaned footprints:TestPoint_Pad_D2.0mm_ValueSilk, B.Cu at (171.2, 138.2)
- added TP23: IO48, cleaned footprints:TestPoint_Pad_D2.0mm_ValueSilk, B.Cu at (168.2, 138.2)
Routing:
- net Net-(U7-IO46): track 0.00 -> 104.6 mm, vias 0 -> 2
- net Net-(U11-IO46): track 104.6 -> 0.00 mm, vias 1 -> 0
- net Net-(U7-IO47): track 0.00 -> 93.0 mm, vias 0 -> 2
- net Net-(U11-IO47): track 93.0 -> 0.00 mm, vias 1 -> 0
- net Net-(U7-IO48): track 0.00 -> 91.2 mm, vias 0 -> 2
- net Net-(U11-IO48): track 91.2 -> 0.00 mm
- net Net-(U7-IO45): track 0.00 -> 87.4 mm, vias 0 -> 2
- net Net-(U11-IO45): track 87.4 -> 0.00 mm, vias 1 -> 0
- net Net-(U7-IO40): track 0.00 -> 76.1 mm, vias 0 -> 2
- net Net-(U11-IO40): track 76.1 -> 0.00 mm, vias 1 -> 0
- net Net-(U7-IO41): track 0.00 -> 72.2 mm, vias 0 -> 2
- net Net-(U11-IO41): track 72.2 -> 0.00 mm, vias 2 -> 0
- net Net-(U7-IO42): track 0.00 -> 68.0 mm, vias 0 -> 2
- net Net-(U11-IO42): track 68.0 -> 0.00 mm, vias 2 -> 0
- net (no net): vias 6 -> 0
