File: electronics/view_base/view_base-backup.kicad_sch (KiCad schematic)
At the start: 279 parts, among them J1 USB_C_Receptacle_USB2.0, J2 A, J3 B, J4 LCD, J5 59453-081110EDHLF, J6 BLDC, J7 SM04B-SRSS-TB(LF)(SN), J8 SM04B-SRSS-TB(LF)(SN), J9 SM04B-SRSS-TB(LF)(SN), Q1 MMBT4403, Q2 BSS138, Q3 BSS138, SW1 RST, SW2 Boot, U1 SN74LV1T34DBV, U10 LP5907MFX-2.8, U11 ESP32-S3-WROOM-1U-N16R8, U12 BQ27427YZFR, U2 MT6701-CT, U3 VEML7700, U4 AMS1117-3.3, U5 USBLC6-2SC6, U6 HX711, U7 MCP73871-2CC, U8 TMC6300, U9 VL53L0CXV0DH_1

Commit message: Initial commit
Parts:
- removed BT1: Battery_Cell, symbol Device:Battery_Cell
- removed C100: 1uF, cleaned footprints:C_0805_2012Metric, symbol Device:C_Small
- removed C96: 10uF, cleaned footprints:C_0805_2012Metric, symbol Device:C_Small
- removed C97: 2.2uF, cleaned footprints:C_0805_2012Metric, symbol Device:C_Small
- removed C98, C99: 4.7uF, cleaned footprints:C_0805_2012Metric, symbol Device:C_Small
- removed D73, D74, D75: LED_Small, symbol Device:LED_Small
- removed R29, R30, R31: 470, symbol Device:R_Small
- removed R32: 10K, symbol Device:R_Small
- removed R33, R35, R36, R37, R38: 10k, symbol Device:R_Small
- removed R34: 1k, symbol Device:R_Small
- removed U12: BQ27427YZFR, Package_BGA:Texas_DSBGA-9_1.62x1.58mm_Layout3x3_P0.5mm, symbol own:BQ27427YZFR
- removed U7: MCP73871-2CC, Package_DFN_QFN:QFN-20-1EP_4x4mm_P0.5mm_EP2.5x2.5mm, symbol Battery_Management:MCP73871-2CC
- TP1, TP10, TP11, TP14, TP15, TP16, TP2, TP24, TP25, TP26, TP27, TP28, TP29, TP3, TP30, TP31, TP32, TP4, TP5, TP6, TP7, TP8, TP9: footprint TestPoint:TestPoint_Pad_D2.0mm -> cleaned footprints:TestPoint_Pad_D2.0mm_ValueSilk
Connections:
- net +4V2 is gone; now on net +5V: U4.3 (Input)
- net +5VUSB is gone; now on net +5V: J1.A4 (VBUS), J1.A9 (VBUS), J1.B4 (VBUS), J1.B9 (VBUS)
- net GND: no longer SW1.2
Other:
- note removed: "BATTERY MANAGEMENT"
- note removed: "FUEL GAUGE"
- note removed: "TODO: Consider a battery with an insert pin"
- note removed: "TODO: add the 4.2 to 5v booster"
- note removed: "TODO: find out if I can actually give this 4.2V"
- note removed: "TODO: look into Prog1 and prog3 values once cell selected"
- note removed: "TODO: swap this for a 2pin connector (with insert detection?)"
- moved on the sheet: C1, C3, C4, C5, J1, R1, R2, TP1, TP2, TP3, TP4, U1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
