File: electronics/view_screen/view_screen.kicad_sch (KiCad schematic)
At the start: 17 parts, among them J2 GC9A01, J6 LCD - FPC, Q1 2N7002

Commit message: Add parts for screen board
Parts:
- J6: LCSC (none) -> C5407791
- Q1: LCSC 2N7002 -> C8545
- R2: LCSC (none) -> C112307
- R3: LCSC (none) -> C22935
Changed lines of the file:
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@@
 (kicad_sch
-	(version 20231120)
+	(version 20250114)
 	(generator "eeschema")
-	(generator_version "8.0")
+	(generator_version "9.0")
 	(paper "A4")
 	(title_block
@@
 		(comment 2 "Original Design by Scott Bezek")
 	)
+	(text "Additional Design by Seedlabs"
+		(exclude_from_sim no)
+		(at 156.21 33.274 0)
+		(effects
+			(font
+				(size 4 4)
+				(thickness 0.4013)
+				(bold yes)
+				(italic yes)
+			)
+			(justify left bottom)
+		)
+	)
+	(text "LCD connector"
+		(exclude_from_sim no)
+		(at 34.29 39.116 0)
+		(effects
+			(font
+				(size 1.27 1.27)
+			)
+		)
+	)
+	(text "Original Design by Scott Bezek"
+		(exclude_from_sim no)
+		(at 26.67 33.782 0)
+		(effects
+			(font
+				(size 4 4)
+				(thickness 0.4013)
+				(bold yes)
+				(italic yes)
+			)
+			(justify left bottom)
+		)
+	)
 	(junction
 		(at 64.77 57.15)
@@
 		)
 	)
-	(text "Additional Design by Seedlabs"
-		(exclude_from_sim no)
-		(at 156.21 33.274 0)
-		(effects
-			(font
-				(size 4 4)
-				(thickness 0.4013)
-				(bold yes)
-				(italic yes)
-			)
-			(justify left bottom)
-		)
-	)
-	(text "LCD connector"
-		(exclude_from_sim no)
-		(at 34.29 39.116 0)
-		(effects
-			(font
-				(size 1.27 1.27)
-			)
-		)
-	)
-	(text "Original Design by Scott Bezek"
-		(exclude_from_sim no)
-		(at 26.67 33.782 0)
-		(effects
-			(font
-				(size 4 4)
-				(thickness 0.4013)
-				(bold yes)
-				(italic yes)
-			)
-			(justify left bottom)
-		)
-	)
 	(label "BACKLIGHT_EN"
 		(at 29.21 86.36 0)
-		(fields_autoplaced yes)
 		(effects
 			(font
@@
 	(label "MOSI"
 		(at 86.36 72.39 0)
-		(fields_autoplaced yes)
 		(effects
 			(font
@@
 	(label "GND"
 		(at 49.53 58.42 180)
-		(fields_autoplaced yes)
 		(effects
 			(font
@@
 	(label "VDD"
 		(at 86.36 52.07 0)
-		(fields_autoplaced yes)
 		(effects
 			(font
@@
 	(label "VDD"
 		(at 71.12 90.17 0)
-		(fields_autoplaced yes)
 		(effects
 			(font
@@
 	(label "DC"
 		(at 49.53 63.5 180)
-		(fields_autoplaced yes)
 		(effects
 			(font
@@
 	(label "nRESET"
 		(at 49.53 73.66 180)
-		(fields_autoplaced yes)
 		(effects
 			(font
@@
 	(label "LEDK"
 		(at 53.34 86.36 0)
-		(fields_autoplaced yes)
 		(effects
 			(font
@@
 	(label "nCS"
 		(at 160.02 63.5 0)
-		(fields_autoplaced yes)
 		(effects
 			(font
@@
 	(label "DC"
 		(at 86.36 57.15 0)
-		(fields_autoplaced yes)
 		(effects
 			(font
@@
 	(label "LEDA"
 		(at 49.53 53.34 180)
-		(fields_autoplaced yes)
 		(effects
 			(font
@@
 	(label "GND"
 		(at 49.53 76.2 180)
-		(fields_autoplaced yes)
 		(effects
 			(font
@@
 	(label "MOSI"
 		(at 49.53 71.12 180)
-		(fields_autoplaced yes)
 		(effects
 			(font
@@
 	(label "SCK"
 		(at 160.02 55.88 0)
-		(fields_autoplaced yes)
 		(effects
 			(font
@@
 	(label "VDD"
 		(at 59.69 49.53 0)
-		(fields_autoplaced yes)
 		(effects
 			(font
@@
 	(label "GND"
 		(at 49.53 60.96 180)
-		(fields_autoplaced yes)
 		(effects
 			(font
@@
 	(label "GND"
 		(at 86.36 49.53 0)
-		(fields_autoplaced yes)
 		(effects
 			(font
@@
 	(label "BACKLIGHT_EN"
 		(at 86.36 54.61 0)
-		(fields_autoplaced yes)
 		(effects
 			(font
@@
 	(label "BACKLIGHT_EN"
 		(at 160.02 60.96 0)
-		(fields_autoplaced yes)
 		(effects
 			(font
@@
 	(label "nCS"
 		(at 86.36 67.31 0)
-		(fields_autoplaced yes)
 		(effects
 			(font
@@
 	(label "LEDK"
 		(at 49.53 50.8 180)
-		(fields_autoplaced yes)
 		(effects
 			(font
@@
 	(label "SCK"
 		(at 49.53 68.58 180)
-		(fields_autoplaced yes)
 		(effects
 			(font
@@
 	(label "VDD"
 		(at 160.02 48.26 0)
-		(fields_autoplaced yes)
 		(effects
 			(font
@@
 	(label "GND"
 		(at 160.02 50.8 0)
-		(fields_autoplaced yes)
 		(effects
 			(font
@@
 	(label "VDD"
 		(at 49.53 55.88 180)
-		(fields_autoplaced yes)
 		(effects
 			(font
@@
 	(label "DC"
 		(at 160.02 66.04 0)
-		(fields_autoplaced yes)
 		(effects
 			(font
@@
 	(label "MOSI"
 		(at 160.02 58.42 0)
-		(fields_autoplaced yes)
 		(effects
 			(font
@@
 	(label "LEDA"
 		(at 71.12 113.03 0)
-		(fields_autoplaced yes)
 		(effects
 			(font
@@
 	(label "SCK"
 		(at 86.36 69.85 0)
-		(fields_autoplaced yes)
 		(effects
 			(font
@@
 	(label "nRESET"
 		(at 86.36 74.93 0)
-		(fields_autoplaced yes)
 		(effects
 			(font
@@
 	(label "nCS"
 		(at 49.53 66.04 180)
-		(fields_autoplaced yes)
 		(effects
 			(font
@@
 	(label "nRESET"
 		(at 160.02 53.34 0)
-		(fields_autoplaced yes)
 		(effects
 			(font
@@
 	(label "GND"
 		(at 49.53 48.26 180)
-		(fields_autoplaced yes)
 		(effects
 			(font
@@
 			)
 		)
-		(property "LCSC" "2N7002"
+		(property "LCSC" "C8545"
 			(at 54.61 100.33 0)
 			(effects
@@
 			)
 		)
+		(property "LCSC" "C22935"
+			(at 44.45 107.95 0)
+			(effects
+				(font
+					(size 1.27 1.27)
+				)
+				(hide yes)
+			)
+		)
 		(pin "1"
 		)
@@
 		)
 		(property "Mouser" "652-CR0603FX-22R0ELF"
+			(at 77.47 101.6 0)
+			(effects
+				(font
+					(size 1.27 1.27)
+				)
+				(hide yes)
+			)
+		)
+		(property "LCSC" "C112307"
 			(at 77.47 101.6 0)
 			(effects
@@
 			)
 		)
+		(property "LCSC" "C5407791"
+			(at 181.61 58.42 0)
+			(effects
+				(font
+					(size 1.27 1.27)
+				)
+				(hide yes)
+			)
+		)
 		(pin "1"
 		)
@@
 		)
 	)
+	(embedded_fonts no)
 )
